Commit message: Update robot description for Melodic
Change laser macro origin roll arg name from "or" to "oroll". "or" seems to be reserved now
Merge accurate model in as a param to the main model
Add some xacro: namespacing to silence warnings

File: gizmo_description/urdf/robots/gizmo/robot.urdf.xacro (robot description, xacro)
@@ -1,30 +1,33 @@
 <?xml version="1.0"?>
 <robot name="gizmo" xmlns:xacro="http://ros.org/wiki/xacro">
+  <xacro:arg name="accurate" default="True" />
   <xacro:include filename="$(find gizmo_description)/urdf/common_properties.urdf.xacro"/>
   <xacro:include filename="$(find gizmo_description)/urdf/sensors/2d_laser.urdf.xacro"/>
   <xacro:include filename="$(find gizmo_description)/urdf/materials.urdf.xacro" />
   <xacro:include filename="$(find gizmo_description)/urdf/sensors/upward_camera.urdf.xacro"/>
-  <xacro:include filename="$(find gizmo_description)/urdf/robots/gizmo/gazebo.urdf.xacro"/>
+  <xacro:include filename="$(find gizmo_description)/urdf/robots/gizmo/gazebo.urdf.xacro">
+    <xacro:arg name="accurate" value="$(arg accurate)"/>
+  </xacro:include>
   <xacro:include filename="$(find gizmo_description)/urdf/robots/gizmo/base.urdf.xacro" />
   <xacro:include filename="$(find gizmo_description)/urdf/robots/gizmo/body.urdf.xacro"/>
   <xacro:include filename="$(find gizmo_description)/urdf/robots/gizmo/head.urdf.xacro"/>
-  <property name="upward_cam_x_loc" value="0.061" />
-  <property name="upward_cam_y_loc" value="-0.032" />
-  <property name="upward_cam_z_loc" value="0.015" />
-  <property name="upward_cam_r_ori" value="0" />
-  <property name="upward_cam_p_ori" value="0" />
-  <property name="upward_cam_y_ori" value="0" />
-  <property name="mount_px" value="0.00022" />
-  <property name="mount_py" value="0.0" />
-  <property name="mount_pz" value="0.08510" />
-  <property name="mount_or" value="${M_PI}" />
-  <property name="mount_op" value="${M_PI}" />
-  <property name="mount_oy" value="${M_PI}" />
-  <property name="laser_px" value="0.0" />
-  <property name="laser_py" value="0.0" />
-  <property name="laser_pz" value="0.155" />
-  <property name="laser_or" value="0" />
-  <property name="laser_op" value="0" />
-  <property name="laser_oy" value="0" />
+  <xacro:property name="upward_cam_x_loc" value="0.061" />
+  <xacro:property name="upward_cam_y_loc" value="-0.032" />
+  <xacro:property name="upward_cam_z_loc" value="0.015" />
+  <xacro:property name="upward_cam_r_ori" value="0" />
+  <xacro:property name="upward_cam_p_ori" value="0" />
+  <xacro:property name="upward_cam_y_ori" value="0" />
+  <xacro:property name="mount_px" value="0.00022" />
+  <xacro:property name="mount_py" value="0.0" />
+  <xacro:property name="mount_pz" value="0.08510" />
+  <xacro:property name="mount_or" value="${M_PI}" />
+  <xacro:property name="mount_op" value="${M_PI}" />
+  <xacro:property name="mount_oy" value="${M_PI}" />
+  <xacro:property name="laser_px" value="0.0" />
+  <xacro:property name="laser_py" value="0.0" />
+  <xacro:property name="laser_pz" value="0.155" />
+  <xacro:property name="laser_or" value="0" />
+  <xacro:property name="laser_op" value="0" />
+  <xacro:property name="laser_oy" value="0" />
   <base/>
   <body />

File: gizmo_description/urdf/robots/p3/robot.urdf.xacro (robot description, xacro)
@@ -11,23 +11,23 @@
   <xacro:include filename="$(find gizmo_description)/urdf/robots/gizmo/body.urdf.xacro"/>
   <xacro:include filename="$(find gizmo_description)/urdf/robots/gizmo/head.urdf.xacro"/>
-  <property name="upward_cam_x_loc" value="0.076" />
-  <property name="upward_cam_y_loc" value="0.0324" />
-  <property name="upward_cam_z_loc" value="0.015" />
-  <property name="upward_cam_r_ori" value="0" />
-  <property name="upward_cam_p_ori" value="0" />
-  <property name="upward_cam_y_ori" value="0" />
-  <property name="mount_px" value="0.00022" />
-  <property name="mount_py" value="0.0" />
-  <property name="mount_pz" value="0.08510" />
-  <property name="mount_or" value="${M_PI}" />
-  <property name="mount_op" value="${M_PI}" />
-  <property name="mount_oy" value="${M_PI}" />
+  <xacro:property name="upward_cam_x_loc" value="0.076" />
+  <xacro:property name="upward_cam_y_loc" value="0.0324" />
+  <xacro:property name="upward_cam_z_loc" value="0.015" />
+  <xacro:property name="upward_cam_r_ori" value="0" />
+  <xacro:property name="upward_cam_p_ori" value="0" />
+  <xacro:property name="upward_cam_y_ori" value="0" />
+  <xacro:property name="mount_px" value="0.00022" />
+  <xacro:property name="mount_py" value="0.0" />
+  <xacro:property name="mount_pz" value="0.08510" />
+  <xacro:property name="mount_or" value="${M_PI}" />
+  <xacro:property name="mount_op" value="${M_PI}" />
+  <xacro:property name="mount_oy" value="${M_PI}" />
   <!-- Depth sensor or Hokuyo -->
-  <property name="laser_px" value="0.109" />
-  <property name="laser_py" value="0.0" />
-  <property name="laser_pz" value="0.175" />
-  <property name="laser_or" value="0" />
-  <property name="laser_op" value="0" />
-  <property name="laser_oy" value="0" />
+  <xacro:property name="laser_px" value="0.109" />
+  <xacro:property name="laser_py" value="0.0" />
+  <xacro:property name="laser_pz" value="0.175" />
+  <xacro:property name="laser_or" value="0" />
+  <xacro:property name="laser_op" value="0" />
+  <xacro:property name="laser_oy" value="0" />
   <base/>
   <body />

File: gizmo_description/urdf/sensors/2d_laser.urdf.xacro (robot description, xacro)
@@ -2,7 +2,7 @@
 <robot name="2D_laser" xmlns:xacro="http://ros.org/wiki/xacro">
   <xacro:include filename="$(find gizmo_description)/urdf/sensors/gazebo.urdf.xacro"/>
-  <xacro:macro name="laser_2D" params="parent suffix px py pz or op oy">
+  <xacro:macro name="laser_2D" params="parent suffix px py pz oroll op oy">
     <joint name="laser_joint${suffix}" type="fixed">
-      <origin xyz="${px} ${py} ${pz}" rpy="${or} ${op} ${oy}" />
+      <origin xyz="${px} ${py} ${pz}" rpy="${oroll} ${op} ${oy}" />
       <parent link="${parent}" />
       <child link="hokuyo_laser_link${suffix}" />
@@ -29,9 +29,9 @@
   </xacro:macro>
   <xacro:macro name="single_2D_laser" params="parent">
-    <laser_2D parent="${parent}" suffix="" px="${laser_px}" py="${laser_py}" pz="${laser_pz}" or="${laser_or}" op="${laser_op}" oy="${laser_oy}"/>
+    <laser_2D parent="${parent}" suffix="" px="${laser_px}" py="${laser_py}" pz="${laser_pz}" oroll="${laser_or}" op="${laser_op}" oy="${laser_oy}"/>
   </xacro:macro>
   <xacro:macro name="dual_2D_lasers" params="parent">
-    <laser_2D parent="${parent}" suffix="" px="${laser_px}" py="${laser_py}" pz="${laser_pz}" or="${laser_or}" op="${laser_op}" oy="${laser_oy}"/>
-    <laser_2D parent="${parent}" suffix="2" px="${laser2_px}" py="${laser2_py}" pz="${laser2_pz}" or="${laser2_or}" op="${laser2_op}" oy="${laser2_oy}"/>
+    <laser_2D parent="${parent}" suffix="" px="${laser_px}" py="${laser_py}" pz="${laser_pz}" oroll="${laser_or}" op="${laser_op}" oy="${laser_oy}"/>
+    <laser_2D parent="${parent}" suffix="2" px="${laser2_px}" py="${laser2_py}" pz="${laser2_pz}" oroll="${laser2_or}" op="${laser2_op}" oy="${laser2_oy}"/>
   </xacro:macro>
 </robot>

File: gizmo_description/urdf/sensors/gazebo.urdf.xacro (robot description, xacro)
@@ -16,5 +16,10 @@
           <clip>
             <near>0.05</near>
-            <far>8.0</far>
+            <xacro:if value="$(arg accurate)">
+                <far>2.43</far>
+            </xacro:if>
+            <xacro:if value="${not $(arg accurate)}">
+                <far>8.0</far>
+            </xacro:if>
           </clip>
         </camera>
@@ -57,5 +62,10 @@
 	  <range>
 	    <min>0.1</min>
-	    <max>15.0</max>
+        <xacro:if value="$(arg accurate)">
+            <max>2.43</max>
+        </xacro:if>
+        <xacro:if value="${not $(arg accurate)}">
+            <max>8.0</max>
+        </xacro:if>
 	    <resolution>0.01</resolution>
 	  </range>
